File: schematics/fet_high_side_switch.sch (EAGLE design)
At the start: 3 parts, among them Q1 MOSFET-NCHANNEL2N7000, Q2 MOSFET-PCHANNELSMD

Commit message: Numerous errata
Connections:
- net VCC renamed +12V
Changed lines of the file:
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@@
 <parts>
 <part name="GND1" library="supply1" deviceset="GND" device=""/>
-<part name="P+1" library="supply1" deviceset="VCC" device=""/>
 <part name="Q1" library="SparkFun-DiscreteSemi" deviceset="MOSFET-NCHANNEL" device="2N7000" value=""/>
 <part name="Q2" library="SparkFun-DiscreteSemi" deviceset="MOSFET-PCHANNEL" device="SMD" value=""/>
 <part name="R1" library="SparkFun-Passives" deviceset="RESISTOR" device="0402-RES" value="100k"/>
+<part name="P+1" library="supply1" deviceset="+12V" device=""/>
 </parts>
 <sheets>
@@
 <instances>
 <instance part="GND1" gate="1" x="20.32" y="-7.62"/>
-<instance part="P+1" gate="VCC" x="20.32" y="30.48"/>
 <instance part="Q1" gate="G$1" x="20.32" y="2.54"/>
 <instance part="Q2" gate="G$1" x="27.94" y="25.4" rot="MR90"/>
 <instance part="R1" gate="G$1" x="20.32" y="17.78" rot="R90"/>
+<instance part="P+1" gate="1" x="20.32" y="30.48"/>
 </instances>
 <busses>
 </busses>
 <nets>
-<net name="VCC" class="0">
-<segment>
-<pinref part="P+1" gate="VCC" pin="VCC"/>
-<pinref part="R1" gate="G$1" pin="2"/>
-<wire x1="20.32" y1="27.94" x2="20.32" y2="25.4" width="0.1524" layer="91"/>
-<pinref part="Q2" gate="G$1" pin="S"/>
-<wire x1="20.32" y1="25.4" x2="20.32" y2="22.86" width="0.1524" layer="91"/>
-<wire x1="22.86" y1="25.4" x2="20.32" y2="25.4" width="0.1524" layer="91"/>
-<junction x="20.32" y="25.4"/>
-</segment>
-</net>
 <net name="N$1" class="0">
 <segment>
@@
 </segment>
 </net>
+<net name="+12V" class="0">
+<segment>
+<pinref part="R1" gate="G$1" pin="2"/>
+<wire x1="20.32" y1="27.94" x2="20.32" y2="25.4" width="0.1524" layer="91"/>
+<pinref part="Q2" gate="G$1" pin="S"/>
+<wire x1="20.32" y1="25.4" x2="20.32" y2="22.86" width="0.1524" layer="91"/>
+<wire x1="22.86" y1="25.4" x2="20.32" y2="25.4" width="0.1524" layer="91"/>
+<junction x="20.32" y="25.4"/>
+<pinref part="P+1" gate="1" pin="+12V"/>
+</segment>
+</net>
