File: schematics/fet_level_shifter.sch (EAGLE design)
At the start: 3 parts, among them Q1 MOSFET-NCHANNEL2N7000

Commit message: Numerous errata
Other:
- note added: "D"
- note added: "G"
- note added: "S"
Changed lines of the file:
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@@
 <sheet>
 <plain>
+<text x="20.828" y="21.844" size="1.778" layer="91">G</text>
+<text x="15.748" y="18.288" size="1.778" layer="91">S</text>
+<text x="23.368" y="18.288" size="1.778" layer="91">D</text>
 </plain>
 <instances>
